File: softstart.kicad_sch (KiCad schematic)
At the start: 17 parts, among them J1 Conn_01x02, Q1 IRF100B201, Q2 IRF100B201, U1 L78L15_TO92, U2 LM393

Commit message: fix comp output
Parts:
- C3: value 2.2n -> 100n
- R3, R4: value 330 -> 1k
Connections:
- net +15V: now also R3.2
- net at R3.1, U2.1: now also C3.1, Q1.1 (G), R5.1
- net at RV1.2, U2.3 (+): no longer C3.1
Other:
- note added: "NTC protection"
- note added: "comparator circuit"
- note added: "power supply"
- note added: "reference voltage"
- moved on the sheet: R3, R4
